Commit message: caster wheels in urdf, ekf yaml, and update launch

File: ros_ws/src/fetch_description/robots/fetch.urdf (robot description, URDF)
Before this commit: robot fetch, 26 links, 25 joints
Links:
- added link imu_link; collision box size=0.1 0.1 0.1; visual box size=0.1 0.1 0.1
Joints:
- added joint imu_joint: type fixed, parent base_link, child imu_link, origin xyz=0 0 0.2878

Commit message: fetch nav param and launch file updates

File: ros_ws/src/fetch_description/robots/fetch.urdf (robot description, URDF)
Before this commit: robot fetch, 27 links, 26 joints
Joints:
- joint laser_joint: origin xyz=0.235 0 0.2878 rpy=3.14159265359 0 0 -> xyz=0.22 0 0.2878 rpy=3.14159265359 0 0

Commit message: Nav2 integrated. Bug with two bot configs switch

File: ros_ws/src/fetch_description/robots/fetch.urdf (robot description, URDF)
Before this commit: robot fetch, 27 links, 26 joints
Joints:
- joint l_wheel_joint: limit effort=8.85 velocity=17.4 -> (none)
- joint r_wheel_joint: limit effort=8.85 velocity=17.4 -> (none)

Commit message: urdf, launch, and ekf updates

File: ros_ws/src/fetch_description/robots/fetch.urdf (robot description, URDF)
Before this commit: robot fetch, 27 links, 26 joints
Links:
- link l_wheel_link: geometry collision sphere radius=0.06033; visual mesh filename=package://fetch_description/meshes/l_wheel_link.STL
- link r_wheel_link: geometry collision sphere radius=0.06033; visual mesh filename=package://fetch_description/meshes/r_wheel_link.STL
Joints:
- joint elbow_flex_joint: origin xyz=0.133 0 0 rpy=0 0 0 -> xyz=0.133 0 0 rpy=0 2.0 0; type revolute -> fixed
- joint forearm_roll_joint: type continuous -> fixed
- joint head_pan_joint: type revolute -> fixed
- joint head_tilt_joint: type revolute -> fixed
- joint l_gripper_finger_joint: type prismatic -> fixed
- joint r_gripper_finger_joint: type prismatic -> fixed
- joint shoulder_lift_joint: axis 0 1 0 -> 0 0.9 0; origin xyz=0.117 0 0.0599999999999999 rpy=0 0 0 -> xyz=0.117 0 0.0599999999999999 rpy=0 1.39 0; type revolute -> fixed
- joint shoulder_pan_joint: origin xyz=0.119525 0 0.34858 rpy=0 0 0 -> xyz=0.119525 0 0.34858 rpy=0 0 1.9; type revolute -> fixed
- joint torso_lift_joint: type prismatic -> fixed
- joint upperarm_roll_joint: type continuous -> fixed
- joint wrist_flex_joint: origin xyz=0.1245 0 0 rpy=0 0 0 -> xyz=0.1245 0 0 rpy=0 1.5 0; type revolute -> fixed
- joint wrist_roll_joint: type continuous -> fixed
